File: HX711.kicad_pcb (KiCad board)
At the start: 2 copper layers, 30 x 25 mm, 9 parts, among them J1 Load-Cell, J2 MCU, J3 RATE, U1 HX711

Commit message: test kicad pcb change
Parts:
- moved H1 5.00 mm to (133.0, 98.0)
- moved J1 0.50 mm to (127.5, 103.0)
Routing:
- net GND: track 14.5 -> 17.1 mm, vias 8 -> 9
Changed lines of the file:
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@@
 		(capping no)
 		(filling no)
-		(zone_defaults)
 		(pcbplotparams
 			(layerselection 0x00000000_00000000_55555555_5755f5ff)
@@
 	(footprint "MountingHole:MountingHole_2.2mm_M2"
 		(layer "F.Cu")
-		(at 128 98)
+		(at 133 98)
 		(descr "Mounting Hole 2.2mm, M2, no annular, generated by kicad-footprint-generator mountinghole.py")
 		(tags "mountinghole M2")
@@
 	(footprint "Connector_PinHeader_2.54mm:PinHeader_1x04_P2.54mm_Vertical"
 		(layer "F.Cu")
-		(at 128 103)
+		(at 127.5 103)
 		(descr "Through hole straight pin header, 1x04, 2.54mm pitch, single row")
 		(tags "Through hole pin header THT 1x04 2.54mm single row")
@@
 	)
 	(segment
+		(start 135 106)
+		(end 135.5 105.5)
+		(width 0.5)
+		(layer "F.Cu")
+		(net "GND")
+	)
+	(segment
 		(start 149 100)
 		(end 149.5 100.5)
@@
 	)
 	(segment
+		(start 137.05 107.08)
+		(end 137.05 107.05)
+		(width 0.5)
+		(layer "F.Cu")
+		(net "GND")
+	)
+	(segment
 		(start 143.04 104.54)
 		(end 143.5 105)
@@
 	)
 	(segment
+		(start 135.5 107)
+		(end 135 107.5)
+		(width 0.5)
+		(layer "F.Cu")
+		(net "GND")
+	)
+	(segment
 		(start 140.4 118.5)
 		(end 141.5 118.5)
@@
 	)
 	(segment
-		(start 135 106)
-		(end 135.19 105.81)
-		(width 0.5)
-		(layer "F.Cu")
-		(net "GND")
-	)
-	(segment
 		(start 142 104.54)
 		(end 143.04 104.54)
@@
 	)
 	(segment
+		(start 136.74 105.5)
+		(end 137.05 105.81)
+		(width 0.5)
+		(layer "F.Cu")
+		(net "GND")
+	)
+	(segment
 		(start 140.05 114)
 		(end 141 114)
@@
 	)
 	(segment
+		(start 135.5 105.5)
+		(end 136.74 105.5)
+		(width 0.5)
+		(layer "F.Cu")
+		(net "GND")
+	)
+	(segment
 		(start 147 100)
 		(end 149 100)
@@
 	)
 	(segment
-		(start 135.19 105.81)
-		(end 137.05 105.81)
+		(start 137 107)
+		(end 135.5 107)
 		(width 0.5)
 		(layer "F.Cu")
@@
 		(start 140.05 116)
 		(end 141 116)
+		(width 0.5)
+		(layer "F.Cu")
+		(net "GND")
+	)
+	(segment
+		(start 137.05 107.05)
+		(end 137 107)
 		(width 0.5)
 		(layer "F.Cu")
@@
 		(size 0.6)
 		(drill 0.3)
+		(layers "F.Cu" "B.Cu")
+		(net "GND")
+	)
+	(via
+		(at 135 107.5)
+		(size 0.6)
+		(drill 0.3)

Commit message: correct test on a branch
Parts:
- moved H1 5.00 mm to (128.0, 98.0)
Changed lines of the file:
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@@
 	(footprint "MountingHole:MountingHole_2.2mm_M2"
 		(layer "F.Cu")
-		(at 133 98)
+		(at 128 98)
 		(descr "Mounting Hole 2.2mm, M2, no annular, generated by kicad-footprint-generator mountinghole.py")
 		(tags "mountinghole M2")
@@
 	)
 	(segment
-		(start 137.05 107.08)
-		(end 137.05 107.05)
-		(width 0.5)
-		(layer "F.Cu")
-		(net "GND")
-	)
-	(segment
 		(start 143.04 104.54)
 		(end 143.5 105)
@@
 	)
 	(segment
-		(start 135.5 107)
-		(end 135 107.5)
-		(width 0.5)
-		(layer "F.Cu")
-		(net "GND")
-	)
-	(segment
 		(start 140.4 118.5)
 		(end 141.5 118.5)
@@
 	)
 	(segment
+		(start 135.42 107.08)
+		(end 135 107.5)
+		(width 0.5)
+		(layer "F.Cu")
+		(net "GND")
+	)
+	(segment
 		(start 131 105.5)
 		(end 130.96 105.54)
@@
 	)
 	(segment
+		(start 137.05 107.08)
+		(end 135.42 107.08)
+		(width 0.5)
+		(layer "F.Cu")
+		(net "GND")
+	)
+	(segment
 		(start 147 100)
 		(end 149 100)
@@
 	)
 	(segment
-		(start 137 107)
-		(end 135.5 107)
-		(width 0.5)
-		(layer "F.Cu")
-		(net "GND")
-	)
-	(segment
 		(start 140.05 116)
 		(end 141 116)
 		(width 0.5)
 		(layer "F.Cu")
-		(net "GND")
-	)
-	(segment
-		(start 137.05 107.05)
-		(end 137 107)
-		(width 0.5)
-		(layer "F.Cu")
